File: Hardware/ESP32_Motor_Controller/ESP32_Motor_Controller.kicad_sch (KiCad schematic)
At the start: 0 parts

Commit message: PCB_V2
Other:
- company: APeleV -> ANGEL PELEGRY VELASCO
Changed lines of the file:
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@@
 	(title_block
 		(title "CONTROLLER")
-		(date "2025-04-04")
-		(company "APeleV")
+		(date "2026-04-07")
+		(rev "2")
+		(company "ANGEL PELEGRY VELASCO")
 	)
 	(sheet
