File: Hardware/ESP32_Motor_Controller/ESP32_Motor_Controller.kicad_pcb (KiCad board)
At the start: 2 copper layers, 65 x 56.4 mm, 162 parts, among them IC501 MT6701CT-AKD, J101 XT30PW-M, J102 XT30PW-M, J501 Hall Encoder, J502 CAN1, J503 CAN2, Q101 IRFH7440TRPBF, Q401 IRFH7440TRPBF, Q402 IRFH7440TRPBF, Q403 IRFH7440TRPBF, Q404 IRFH7440TRPBF, Q405 IRFH7440TRPBF, Q406 IRFH7440TRPBF, SW1 TS-1088-AR02016, SW2 TS-1088-AR02016, U2 TLV75733PDBV, U301 DRV8302DCAR, U501 BMI270, U502 MCP2551-I_SN

Commit message: PCB Layout Update
Parts:
- added C508: 0.1uF, Capacitor_SMD:C_0402_1005Metric, F.Cu at (201.4, 77.2)
- added R509: 10k, Resistor_SMD:R_0402_1005Metric, F.Cu at (197.9, 77.2)
- added TH1: NTC 10k, Resistor_SMD:R_0603_1608Metric, F.Cu at (198.0, 80.0)
- C114, C115, Q401, Q402, Q403, Q404, Q405, Q406, R405, R408, U2: moved to B.Cu
- C502: footprint Capacitor_SMD:C_0603_1608Metric -> Capacitor_SMD:C_0402_1005Metric
- JP1: value SOLDER-RPP -> SOLDER - RPP
- JP3: moved to F.Cu
- moved Q405 192.7 mm to (71.9, 80.9), turned to 90 degrees
- moved Q406 192.6 mm to (71.9, 88.4), turned to 90 degrees
- moved Q404 185.5 mm to (78.2, 88.4), turned to 90 degrees
- moved Q403 185.5 mm to (78.3, 81.0), turned to 90 degrees
- moved Q401 179.3 mm to (84.6, 81.0), turned to 90 degrees
- moved Q402 179.3 mm to (84.6, 88.4), turned to 90 degrees
- moved R408 173.8 mm to (77.0, 94.4), turned to 180 degrees
- moved R405 165.1 mm to (85.5, 94.4)
- moved C115 37.8 mm to (138.3, 60.6)
- moved U2 32.4 mm to (138.5, 63.5), turned to -90 degrees
- moved C107 29.8 mm to (201.6, 56.7)
- moved C112 29.8 mm to (206.0, 56.7)
- moved C104 29.8 mm to (201.6, 47.6)
- moved C105 29.8 mm to (201.6, 50.6)
- moved C106 29.8 mm to (201.6, 53.7)
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Connections:
- net CAN_H renamed CAN_P
- net CAN_L renamed CAN_N
- MCU1 pad 11: unconnected-(MCU1-GPIO18/U1RXD/ADC2_CH7/CLK_OUT3-Pad11) -> MAG_CSN
- MCU1 pad 23: MAG_CSN -> MAG_CLK
- MCU1 pad 31: MAG_CLK -> NTC
Routing:
- net MAG_PUSH: track 0.00 -> 25.9 mm, vias 0 -> 1
- net MAG_DO: track 0.00 -> 23.6 mm, vias 0 -> 1
- net MAG_CLK: track 0.00 -> 21.8 mm, vias 0 -> 1
- net MAG_CSN: track 0.00 -> 8.87 mm, vias 0 -> 1
- net AGND: track 0.00 -> 6.42 mm, vias 0 -> 1
- net CAN_N: track 0.00 -> 4.86 mm
- net CAN_P: track 0.00 -> 4.84 mm
- net 3V3: track 0.00 -> 2.68 mm
Other:
- board text added: "CAN"
- board text added: "PVDD"

Commit message: Update Layout
Parts:
- removed TP1: GND, TestPoint:TestPoint_Pad_D1.0mm
- removed TP10: CAN_TX, TestPoint:TestPoint_Pad_D1.0mm
- removed TP11: CAN_RX, TestPoint:TestPoint_Pad_D1.0mm
- removed TP12: BMI_SCK, TestPoint:TestPoint_Pad_D1.0mm
- removed TP13: 5V, TestPoint:TestPoint_Pad_D1.0mm
- removed TP14: PVDD, TestPoint:TestPoint_Pad_D1.0mm
- removed TP15: BMI_SDI, TestPoint:TestPoint_Pad_D1.0mm
- removed TP16: BMI_SDO, TestPoint:TestPoint_Pad_D1.0mm
- removed TP17: MAG_CLK, TestPoint:TestPoint_Pad_D1.0mm
- removed TP18: MAG_CSN, TestPoint:TestPoint_Pad_D1.0mm
- removed TP19: MAG_DO, TestPoint:TestPoint_Pad_D1.0mm
- removed TP2: A_SENSE, TestPoint:TestPoint_Pad_D1.0mm
- removed TP20: VBUS, TestPoint:TestPoint_Pad_D1.0mm
- removed TP21: GND POWER, TestPoint:TestPoint_Pad_D1.0mm
- removed TP3: B_SENSE, TestPoint:TestPoint_Pad_D1.0mm
- removed TP4: C_SENSE, TestPoint:TestPoint_Pad_D1.0mm
- removed TP5: GND, TestPoint:TestPoint_Pad_D1.5mm
- removed TP6: PVDD_SENSE, TestPoint:TestPoint_Pad_D1.0mm
- removed TP7: OC_ADJ, TestPoint:TestPoint_Pad_D1.5mm
- removed TP8: V_SENSE, TestPoint:TestPoint_Pad_D1.5mm
- removed TP9: 3V3, TestPoint:TestPoint_Pad_D1.0mm
- C104, C105, C106, C107, C108, C109, C110, C111, C112, C113, C321, C401, C402, C403, C404, C405, C408, C501, C502, C503, D403, R312, R313, R402, R404, R407, R409, R410, R412, R414, R415, R505: moved to B.Cu
- J501: footprint Connector_JST:JST_PH_S6B-PH-K_1x06_P2.00mm_Horizontal -> Connector_JST:JST_PH_S5B-PH-K_1x05_P2.00mm_Horizontal
- MP1, MP2, MP3: footprint MountingHole:MountingHole_2.5mm -> MountingHole:MountingHole_2.5mm_Pad_Via; moved to B.Cu
- R101, R102: moved to F.Cu
- moved R411 99.3 mm to (137.5, 60.6), turned to 180 degrees
- moved R414 94.4 mm to (134.9, 65.5), turned to 90 degrees
- moved R415 91.2 mm to (134.9, 67.5), turned to 90 degrees
- moved R410 91.1 mm to (135.0, 85.9), turned to 90 degrees
- moved R406 88.7 mm to (135.5, 75.5), turned to 180 degrees
- moved R412 85.9 mm to (143.8, 71.2)
- moved R404 84.3 mm to (137.9, 86.5), turned to 0 degrees
- moved R401 83.3 mm to (135.4, 79.0), turned to 180 degrees
- moved C401 83.3 mm to (143.5, 73.8), turned to 90 degrees
- moved C501 83.0 mm to (184.5, 82.0)
- moved C402 81.6 mm to (137.9, 87.6), turned to 0 degrees
- moved R409 81.0 mm to (135.0, 84.0), turned to 90 degrees
- moved C507 77.6 mm to (180.2, 83.4)
- moved C405 77.6 mm to (143.5, 67.2)
- moved C506 76.0 mm to (182.1, 86.0), turned to -90 degrees
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Connections:
- J101 pad N: PVDD -> /POWER/GND POWER
- J101 pad P: /POWER/GND POWER -> PVDD
- J102 pad N: PVDD -> /POWER/GND POWER
- J102 pad P: /POWER/GND POWER -> PVDD
Routing:
- net CAN_P: track 4.84 -> 59.4 mm, vias 0 -> 1
- net CAN_N: track 4.86 -> 58.1 mm, vias 0 -> 1
- net PVDD: track 0.00 -> 44.4 mm
- net /POWER/GND POWER: track 0.00 -> 26.7 mm
- net 3V3: track 2.68 -> 19.7 mm, vias 0 -> 1
- net BMI_SDO: track 0.00 -> 11.1 mm
- net SH_A: track 0.00 -> 10.5 mm
- net SH_B: track 0.00 -> 9.96 mm
- net SH_C: track 0.00 -> 9.86 mm
- net AGND: track 6.42 -> 14.3 mm, vias 1 -> 5
- net 5V: track 0.00 -> 6.80 mm, vias 0 -> 1
- net BMI_SCK: track 0.00 -> 6.14 mm
- net Net-(D101-K): track 0.00 -> 4.87 mm
- net Net-(JP3-B): track 0.00 -> 2.96 mm
- net /CONTROLLER/EN: track 0.00 -> 2.82 mm
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- added copper zone on B.Cu, net AGND

Commit message: Finished Layout V1
Parts:
- added A: A_SENSE, TestPoint:TestPoint_Pad_D1.0mm, F.Cu at (179.3, 65.4)
- added B: B_SENSE, TestPoint:TestPoint_Pad_D1.0mm, F.Cu at (179.7, 72.7)
- added C: C_SENSE, TestPoint:TestPoint_Pad_D1.0mm, F.Cu at (135.8, 64.7)
- added TP13: 5V, TestPoint:TestPoint_Pad_D1.0mm, B.Cu at (150.4, 100.8)
- added TP6: PVDD_SENSE, TestPoint:TestPoint_Pad_D1.0mm, B.Cu at (151.6, 65.1)
- added TP9: 3V3, TestPoint:TestPoint_Pad_D1.0mm, B.Cu at (141.2, 98.8)
- C303, C308, R411: moved to B.Cu
- D403: moved to F.Cu
- moved C204 31.2 mm to (161.2, 67.4)
- moved SW1 31.2 mm to (157.6, 67.4)
- moved C319 9.53 mm to (149.0, 96.6), turned to -90 degrees
- moved D301 6.39 mm to (144.2, 87.4), turned to 0 degrees
- moved D403 5.65 mm to (159.2, 91.7), turned to 180 degrees
- moved L301 4.13 mm to (144.2, 81.8)
- moved R509 3.42 mm to (177.7, 80.4), turned to 90 degrees
- moved SW2 3.32 mm to (172.4, 95.7)
- moved C316 3.12 mm to (142.2, 85.1), turned to 180 degrees
- moved C318 2.15 mm to (153.5, 86.2), turned to -90 degrees
- moved R306 2.15 mm to (152.5, 86.2), turned to -90 degrees
- moved C508 2.13 mm to (180.4, 80.4), turned to -90 degrees
- moved C205 2.05 mm to (174.0, 97.9), turned to 180 degrees
- moved C320 1.83 mm to (150.3, 72.4), turned to 180 degrees
- moved C308 1.66 mm to (134.1, 72.6), turned to 90 degrees
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Connections:
- IC501 pad 5: MAG_PUSH -> unconnected-(IC501-PUSH-Pad5)
- MCU1 pad 16: NOCTW -> unconnected-(MCU1-GPIO46-Pad16)
- MCU1 pad 21: BMI_SDO -> NTC
- MCU1 pad 24: BMI_SCK -> BMI_SDA
- MCU1 pad 26: MAG_PUSH -> unconnected-(MCU1-GPIO45-Pad26)
- MCU1 pad 28: BMI_CS -> BMI_SCK
- MCU1 pad 29: BMI_SDI -> BMI_CS
- MCU1 pad 31: NTC -> NOCTW
- MCU1 pad 4: INH_A -> INL_C
- MCU1 pad 5: INH_B -> INH_C
- MCU1 pad 6: INH_C -> INL_B
- MCU1 pad 7: INL_A -> INH_B
- MCU1 pad 8: INL_B -> INL_A
- MCU1 pad 9: INL_C -> INH_A
- U501 pad 1: BMI_SDO -> unconnected-(U501-SDO-Pad1)
- U501 pad 14: BMI_SDI -> BMI_SDA
Routing:
- net 3V3: track 19.7 -> 149.9 mm, vias 1 -> 16
- net 5V: track 6.80 -> 132.9 mm, vias 1 -> 10
- net AGND: track 14.3 -> 125.4 mm, vias 5 -> 94
- net B_SENSE: track 0.00 -> 66.5 mm, vias 0 -> 2
- net A_SENSE: track 0.00 -> 64.3 mm, vias 0 -> 2
- net C_SENSE: track 0.00 -> 61.8 mm, vias 0 -> 1
- net NFAULT: track 0.00 -> 49.6 mm, vias 0 -> 2
- net SL_A: track 0.00 -> 47.7 mm, vias 0 -> 3
- net Net-(J501-Pin_3): track 0.00 -> 42.6 mm
- net Net-(J501-Pin_4): track 0.00 -> 42.2 mm
- net Net-(J501-Pin_5): track 0.00 -> 41.9 mm
- net NOCTW: track 0.00 -> 41.5 mm, vias 0 -> 2
- net GL_A: track 0.00 -> 35.8 mm, vias 0 -> 2
- net GAIN: track 0.00 -> 35.6 mm, vias 0 -> 2
- net DC_CAL: track 0.00 -> 35.6 mm, vias 0 -> 2
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- added copper zone on B.Cu, net /POWER/GND POWER
- added copper zone on In2.Cu, net 3V3
- added copper zone on In2.Cu, net 5V
- added copper zone on In1.Cu, net AGND
- added copper zone on B.Cu, net PVDD
- added copper zone on In2.Cu, net PVDD
- added copper zone on B.Cu, net SH_A
- added copper zone on B.Cu, net SH_B
- added copper zone on B.Cu, net SH_C
- added copper zone on B.Cu, net SL_A
- added copper zone on B.Cu, net SL_B
Other:
- outline, holes or cut-outs redrawn
- copper layers 2 -> 4
- board text added: "16V | 40A"
- board text added: "3V3"
- board text added: "5V"
- board text added: "A"
- board text added: "B"
- board text added: "BMI"
- board text added: "BOOT"
- board text added: "C"
- board text added: "DRV"
- board text added: "END-S"
- board text added: "H"
- board text added: "HALL"
- board text added: "L"
- board text added: "MCP 2551"
- board text added: "MT 6701"
- board text added: "PV"
- board text added: "RPP x|+"
- board text added: "RST"
- board text added: "VERSION Nº"
- board text added: "x"
- board text added: "y"
- board text added: "z"

Commit message: Test firmware
Parts:
- added GND: GND, TestPoint:TestPoint_Pad_D1.0mm, B.Cu at (150.4, 103.4)
- renumbered A to TP2, B to TP3, C to TP4
Connections:
- C314 pad 1: Net-(C314-Pad1) -> PVDD
- C315 pad 1: Net-(C314-Pad1) -> PVDD
- U301 pad 53: Net-(C314-Pad1) -> PVDD
- U301 pad 54: Net-(C314-Pad1) -> PVDD
Routing:
- net PVDD: track 59.1 -> 66.6 mm, vias 18 -> 19
- net Net-(C314-Pad1): track 5.77 -> 0.00 mm
- net AGND: track 125.4 -> 127.3 mm

Commit message: PCB V2, CAD V3 & Code
Parts:
- renumbered GND to TP1
Changed lines of the file:
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@@
 		(descr "SMD pad as test Point, diameter 1.0mm")
 		(tags "test point SMD pad")
-		(property "Reference" "GND"
+		(property "Reference" "TP1"
 			(at 2.55 -0.01 0)
 			(layer "B.SilkS")

Commit message: PCB_V2
Parts:
- removed Q101: IRFH7440TRPBF, IRFH7440TRPBF:IRFH7440TRPBF
- removed TP6: PVDD_SENSE, TestPoint:TestPoint_Pad_D1.0mm
- added AV: AVDD, TestPoint:TestPoint_Pad_D1.0mm, F.Cu at (149.9, 66.3)
- added Ext_Cap101: Conn_01x01_Pin, Connector_PinHeader_2.00mm:PinHeader_1x01_P2.00mm_Vertical, F.Cu at (153.3, 89.7)
- added FB: -k, Inductor_SMD:L_0603_1608Metric, B.Cu at (171.5, 100.2)
- added PV: PVDD, TestPoint:TestPoint_Pad_D1.0mm, F.Cu at (133.2, 87.4)
- added Q1: XRS80P06F, XRS80P06F:XRS80P06F, B.Cu at (151.8, 56.1)
- C201, C302, C320: footprint Capacitor_SMD:C_0402_1005Metric -> Capacitor_SMD:C_0603_1608Metric
- C203, C311, C312, C314, C315, C401, C405, C408: footprint Capacitor_SMD:C_0402_1005Metric -> Capacitor_SMD:C_0805_2012Metric
- C313: value 1uF -> 2.2uF; footprint Capacitor_SMD:C_0402_1005Metric -> Capacitor_SMD:C_0805_2012Metric
- C316: footprint Capacitor_SMD:C_0603_1608Metric -> Capacitor_SMD:C_0805_2012Metric
- C317: value 1.6nF -> 1.5nF
- C319: value 49uF -> 47uF
- D301: value B330 -> B360
- ESP 32: renamed from MCU1
- Q401, Q402, Q403, Q404, Q405, Q406: value IRFH7440TRPBF -> FH4008GS; footprint IRFH7440TRPBF:IRFH7440TRPBF -> Package_DFN_QFN:PQFN-8-EP_6x5mm_P1.27mm_Generic
- R202, R205, R301, R302: value 56 -> 56R
- R203: value 150 -> 150R
- R204: value 1100 -> 1100R
- R308: value 10k -> 3.3k
- R309: value 52.3k -> 10k
- R313, R404, R409, R414: value 68k -> 100k
- R504: value 120R -> 121R
- TVS103: footprint Diode_SMD:D_SMA_Handsoldering -> Diode_SMD:D_SMC
- moved R103 13.0 mm to (145.1, 54.6), turned to -90 degrees
- moved D101 8.12 mm to (147.3, 55.8)
- moved C319 8.02 mm to (149.2, 88.6), turned to 90 degrees
- moved C317 4.49 mm to (148.1, 83.4), turned to -90 degrees
- moved C318 4.44 mm to (150.1, 83.4)
- moved R306 4.37 mm to (149.1, 83.5)
- moved R308 3.88 mm to (152.8, 86.0)
- moved R309 3.88 mm to (152.8, 84.5)
- moved C115 2.73 mm to (166.6, 100.2), turned to -90 degrees
- moved C311 2.59 mm to (136.2, 67.2), turned to 90 degrees
- moved C312 2.07 mm to (138.2, 67.2), turned to 90 degrees
- moved R310 1.90 mm to (150.8, 78.6), turned to -90 degrees
- moved C315 1.81 mm to (134.8, 84.2)
- moved C 1.58 mm to (136.2, 63.1)
- moved C313 1.58 mm to (147.0, 67.2)
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- renumbered TP2 to A, TP3 to B, TP4 to C, TP1 to GND, USB101 to USB-C
Connections:
- net Net-(U301-GVDD) renamed /GATE DRIVER/GVDD
- C115 pad 1: 5V -> Net-(U2-EN)
- C313 pad 1: Net-(U301-AGND) -> /GATE DRIVER/AVDD
- D101 pad 1: Net-(D101-K) -> PVDD
- D101 pad 2: AGND -> Net-(D101-A)
- J101 pad N: /POWER/GND POWER -> AGND
- J101 pad P: PVDD -> /POWER/+16 POWER
- J102 pad N: /POWER/GND POWER -> AGND
- J102 pad P: PVDD -> /POWER/+16 POWER
- JP1 pad 1: Net-(JP1-A) -> /POWER/JP1
- JP1 pad 2: PVDD -> /POWER/+16 POWER
- JP2 pad 1: AGND -> /POWER/+16 POWER
- JP2 pad 2: /POWER/GND POWER -> PVDD
- R103 pad 1: Net-(JP1-A) -> Net-(D101-A)
- R103 pad 2: Net-(D101-K) -> AGND
- R309 pad 1: 5V -> 3V3
- TVS103 pad 1: PVDD -> /POWER/+16 POWER
- TVS103 pad 2: /POWER/GND POWER -> AGND
- U2 pad 1: 5V -> Net-(U2-EN)
- U2 pad 3: 5V -> Net-(U2-EN)
- U301 pad 27: Net-(U301-AGND) -> /GATE DRIVER/AVDD
- U301 pad 28: Net-(U301-AGND) -> AGND
- U301 pad 30: SP_2 -> AGND
- U301 pad 32: SP_1 -> AGND
Routing:
- net /POWER/+16 POWER: track 0.00 -> 30.8 mm
- net AGND: track 127.3 -> 154.5 mm, vias 94 -> 164
- net /POWER/GND POWER: track 26.7 -> 0.00 mm
- net PVDD: track 66.6 -> 81.3 mm, vias 19 -> 25
- net 5V: track 132.9 -> 121.1 mm, vias 10 -> 12
- net 3V3: track 149.9 -> 160.2 mm, vias 16 -> 18
- net Net-(U2-EN): track 0.00 -> 7.05 mm
- net /POWER/JP1: track 0.00 -> 6.66 mm
- net Net-(U301-COMP): track 8.91 -> 2.41 mm
- net /GATE DRIVER/AVDD: track 0.00 -> 6.23 mm
- net Net-(U301-VSENSE): track 4.06 -> 8.94 mm
- net Net-(U301-AGND): track 4.31 -> 0.00 mm
- net Net-(D101-K): track 3.89 -> 0.00 mm
- net Net-(D101-A): track 0.00 -> 3.78 mm
- net Net-(JP1-A): track 3.14 -> 0.00 mm
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- added copper zone on B.Cu, net /POWER/JP1
- removed copper zone on B.Cu, net /POWER/GND POWER
Other:
- board text added: "36V | 40A"
- board text added: "RPP +|x"
- board text removed: "16V | 40A"
- board text removed: "RPP x|+"

Commit message: Buck Components Update
Parts:
- C317: value 1.5nF -> 15pF
- C318: value 36pF -> 1nF
- C319: value 47uF -> 22uF
- C506: value 0.1uF -> 1uF
- R306: value 15k -> 86.6k
- R308: value 3.3k -> 10k
- R309: value 10k -> 52.3k
Routing:
- net AGND: vias 164 -> 165
- net 5V: vias 12 -> 11

Commit message: CAN_Bus
MCP2551 is transmitting packets
Parts:
- C319: value 22uF -> 12uH
Connections:
- R309 pad 1: 3V3 -> 5V
Changed lines of the file:
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@@
 			(layers "F.Cu" "F.Mask" "F.Paste")
 			(roundrect_rratio 0.25)
-			(net 101 "3V3")
+			(net 2 "5V")
 			(pintype "passive")
 		)
@@
 			)
 		)
-		(property "Value" "22uF"
+		(property "Value" "12uH"
 			(at 0 1.43 90)
 			(layer "F.Fab")
