File: Hardware/ESP32_Motor_Controller/POWER [1].kicad_sch (KiCad schematic)
At the start: 29 parts, among them J101 XT30PW-M, J102 XT30PW-M, Q101 IRFH7440TRPBF, U2 TLV75733PDBV

Commit message: Update Layout
Connections:
- net GND POWER: now also J101.N, J102.N; no longer J101.P, J102.P
- net PVDD: now also J101.P, J102.P; no longer J101.N, J102.N
Changed lines of the file:
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@@
 		)
 	)
-	(label "GND POWER"
+	(label "+16 POWER"
 		(at 232.41 137.16 180)
 		(effects
@@
 		)
 	)
-	(label "+16 POWER"
+	(label "GND POWER"
 		(at 232.41 139.7 180)
 		(effects

Commit message: PCB_V2
Parts:
- removed Q101: IRFH7440TRPBF, IRFH7440TRPBF:IRFH7440TRPBF, symbol IRFH7440TRPBF_:IRFH7440TRPBF
- removed TP21: GND POWER, TestPoint:TestPoint_Pad_D1.0mm, symbol Connector:TestPoint
- added Ext_Cap101: Conn_01x01_Pin, Connector_PinHeader_2.00mm:PinHeader_1x01_P2.00mm_Vertical, symbol Connector:Conn_01x01_Pin
- added FB1: 600R, Inductor_SMD:L_0603_1608Metric, symbol Device:FerriteBead_Small
- added Q1: XRS80P06F, XRS80P06F:XRS80P06F, symbol XRS80P06F:SI7149DP-T1-GE3
- TVS103: footprint Diode_SMD:D_SMA_Handsoldering -> Diode_SMD:D_SMC
Connections:
- net 5V: now also FB1.1; no longer C115.1, U2.1 (IN), U2.3 (EN)
- net GND: now also J101.N, J102.N, R103.2, TVS103.2; no longer D101.2 (A), JP2.1 (A)
- net PVDD: now also D101.1 (K), JP2.2 (B), Ext_Cap101.1 (Pin_1), Q1.1, Q1.2, Q1.3; no longer J101.P, J102.P, JP1.2 (B), TVS103.1
- net at R103.1: now also D101.2 (A), Q1.4; no longer JP1.1 (A)
- removed net GND POWER: J101.N, J102.N, JP2.2 (B), TVS103.2
- new net: C115.1, FB1.2, U2.1 (IN), U2.3 (EN)
- new net +16 POWER: J101.P, J102.P, JP1.2 (B), JP2.1 (A), TVS103.1
- new net JP1: JP1.1 (A), Q1.5, Q1.6, Q1.7, Q1.8, Q1.9
Other:
- note added: "MOSFET MAX 85V"
- note added: "SMCJ45CA for 36V motors"
- note added: "Solder to PVDD and GND"
- note removed: "DO NOT JOIN GND WITH OTHER GND PLANE"
- note removed: "MAX 18V Protection to MSFT"
- company: (none) -> ANGEL PELEGRY VELASCO
- moved on the sheet: C114, C115, J101, J102, U2
