File: Hardware/ESP32_Motor_Controller/POWER [1].kicad_sch (KiCad schematic)
At the start: 30 parts, among them J101 XT30PW-M, J102 XT30PW-M, Q1 XRS80P06F, U2 TLV75733PDBV

Commit message: Adapted for Main Robot
Parts:
- C104, C105, C106, C107, C108, C109, C110, C111, C112, C113: value 10uF -> 4.7uF
Changed lines of the file:
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@@
 			"NQBVAEgAQQBBAEEAQQBBAEcAQQBEAGYAZgByADAAdQBmAHYAdQB1ADgAVgBKAFgAbAA1AGUAWgBt"
 			"AGEAbQByAEQAeQB3AEIAZwBvAGQAUgA2AFoANABQAE0AZgBiADIAMwB2AGgAdwBvAFcAUwBzAGcA"
-			"QQBBAEEAQQBBAEEAYgBPAGYAKw=="
+			"QQBBAEEAQQBBAEEAYgBPAGYAKwBaAEgAVgAzAGQAMwAvAG8AbwBZAGMAawA1AGcARQBBAEEAQQBB"
+			"AEEAYQBNAEcAdgBmAHYAVwByAG4AagAxADcAbQBnAC8AYgAyAHQAbwArACsATwBDAEQAagBvADQA"
+			"TwBpAFoARgBnAEkAUQBvAGQAeAAxAEYAZABYAGIAMQBxADEAUwBwAHgATQBtAFgASwBsAFAARAB3"
+			"AGMARgBsADUAQQBBAEEAQQBBAEEAQQBhAE0AVwB6AFkAcwBLAFMAawBKAEgARwB5AGQAZQB2AFcA"
+			"cwByAEkAeQBXAFgAbABnAE8AUQBvAGQAeAA3AEYAdQAzAGIAcQBLAGkAZwBwAHgAOAB1AGkAagBq"
+			"ADgAbwBLAEEAdwBBAEEAQQBBAEQAUQBsAEUAYwBmAGYAZABUAFoAKwBkADgAbABRAEYAMQBkADMA"
+			"ZgBmAGYAZgB5ADgAeABEAHkAeABFAG8AZQBNAGcAVABDAGIAVABwADUAOQArAEsAawA2AEcARABS"
+			"AHMAMgBjACsAWgBNAFcAWABrAEEAQQBBAEEAQQBBAEoAbwB5AGUAZgBMAGsAcwBXAFAASABpAHAA"
+			"TgB2AHYAdgBtAG0AbwBhAEYAQgBWAGgANQBZAGkARQBMAEgAUQBlAFQAbQA1AHUAYgBrADUASQBp"
+			"AFQAQgBRAHMAVwA5AE8ANwBkAFcAMQBZAGUAQQBBAEEAQQBBAEkAQwBtAGQATwB2AFcAYgBlAEgA"
+			"QwBoAGUASwBrAHUATABoADQAKwAvAGIAdABrAHUATABBAFUAaABRADYARAB1AEwAVABUAHoAOAAx"
+			"AG0AVQB6AG0AdwAyADcAZAB1AHQAMQAvAC8ALwAwAFMAOAB3AEEAQQBBAEEAQQBBAHQARwBiAHUA"
+			"MwBMAGwAKwBmAG4ANwBtAHcANAA2AE8AagBvADgALwAvAHAAaQBsAGsAZQAwAFUAaABZADQAagBP"
+			"AEgAMwA2ADkASgBvADEAYQA4AFQASgA5AE8AbgBUAFEAMABKAEMAWgBPAFUAQgBBAEEAQQBBAEEA"
+			"RwBqAFEANABNAEcARABiADcALwA5AGQAbgBHAFMAbgBwADUAZQBXAEYAZwBvAEsAdwA4AHMAUQBh"
+			"AEgAagBDAEQAWgBzADIASABEADIANwBGAGwAeAB3AG4ATABJAEEAQQBBAEEAQQBJAEEAcgAvAGYA"
+			"YQAzAHYAMwBWADEAZABUAFUAZgBOAGoAUQAwAEwARgB1ADIAVABHAEkAZQBkAEIAbQBGAGoAaQBQ"
+			"ADQAOABzAHMAdgB4AGMATwBBAGcASQBBAFoATQAyAFoASQB5AGcASQBBAEEAQQBBAEEAMABLADQA"
+			"SgBFAHkAYQBNAEcAVABOAEcAbg=="
 		)
 	)
@@
 			)
 		)
-		(property "Value" "10uF"
+		(property "Value" "4.7uF"
 			(at 255.016 118.872 0)
 			(effects
@@
 			)
 		)
-		(property "Value" "10uF"
+		(property "Value" "4.7uF"
 			(at 192.786 118.872 0)
 			(effects
@@
 			)
 		)
-		(property "Value" "10uF"
+		(property "Value" "4.7uF"
 			(at 183.896 118.872 0)
 			(effects
@@
 			)
 		)
-		(property "Value" "10uF"
+		(property "Value" "4.7uF"
 			(at 175.006 118.872 0)
 			(effects
@@
 			)
 		)
-		(property "Value" "10uF"
+		(property "Value" "4.7uF"
 			(at 245.618 118.872 0)
 			(effects
@@
 			)
 		)
-		(property "Value" "10uF"
+		(property "Value" "4.7uF"
 			(at 228.346 118.872 0)
 			(effects
@@
 			)
 		)
-		(property "Value" "10uF"
+		(property "Value" "4.7uF"
 			(at 210.566 118.872 0)
 			(effects
@@
 			)
 		)
-		(property "Value" "10uF"
+		(property "Value" "4.7uF"
 			(at 219.456 118.872 0)
 			(effects
@@
 			)
 		)
-		(property "Value" "10uF"
+		(property "Value" "4.7uF"
 			(at 237.236 118.872 0)
 			(effects
@@
 			)
 		)
-		(property "Value" "10uF"
+		(property "Value" "4.7uF"
 			(at 201.676 118.872 0)
 			(effects
