File: Hardware/ESP32_Motor_Controller/POWER_MOSFET.kicad_sch (KiCad schematic)
At the start: 38 parts, among them Q401 IRFH7440TRPBF, Q402 IRFH7440TRPBF, Q403 IRFH7440TRPBF, Q404 IRFH7440TRPBF, Q405 IRFH7440TRPBF, Q406 IRFH7440TRPBF

Commit message: Update Layout
Parts:
- MP1, MP2, MP3: footprint MountingHole:MountingHole_2.5mm -> MountingHole:MountingHole_2.5mm_Pad_Via; symbol Mechanical:MountingHole_Pad_MP -> Mechanical:MountingHole_Pad
Connections:
- net SH_A: now also MP1.1; no longer MP1.MP
- net SH_B: now also MP2.1; no longer MP2.MP
- net SH_C: now also MP3.1; no longer MP3.MP
Changed lines of the file:
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@@
 	(wire
 		(pts
+			(xy 119.38 138.43) (xy 119.38 151.13)
+		)
+		(stroke
+			(width 0)
+			(type default)
+		)
+	)
+	(wire
+		(pts
 			(xy 50.8 68.58) (xy 50.8 71.12)
 		)
@@
 	(wire
 		(pts
-			(xy 119.38 138.43) (xy 119.38 151.13)
-		)
-		(stroke
-			(width 0)
-			(type default)
-		)
-	)
-	(wire
-		(pts
 			(xy 50.8 88.9) (xy 50.8 99.06)
 		)
@@
 	)
 	(symbol
-		(lib_id "Mechanical:MountingHole_Pad_MP")
+		(lib_id "Mechanical:MountingHole_Pad")
 		(at 119.38 153.67 180)
 		(unit 1)
@@
 			)
 		)
-		(property "Footprint" "MountingHole:MountingHole_2.5mm"
+		(property "Footprint" "MountingHole:MountingHole_2.5mm_Pad_Via"
 			(at 119.38 153.67 0)
 			(effects
@@
 			)
 		)
-		(property "Description" "Mounting Hole with connection as pad named MP"
+		(property "Description" "Mounting Hole with connection"
 			(at 119.38 153.67 0)
 			(effects
@@
 			)
 		)
-		(pin "MP"
+		(pin "1"
 		)
 		(instances
@@
 	)
 	(symbol
-		(lib_id "Mechanical:MountingHole_Pad_MP")
+		(lib_id "Mechanical:MountingHole_Pad")
 		(at 149.86 153.67 180)
 		(unit 1)
@@
 			)
 		)
-		(property "Footprint" "MountingHole:MountingHole_2.5mm"
+		(property "Footprint" "MountingHole:MountingHole_2.5mm_Pad_Via"
 			(at 149.86 153.67 0)
 			(effects
@@
 			)
 		)
-		(property "Description" "Mounting Hole with connection as pad named MP"
+		(property "Description" "Mounting Hole with connection"
 			(at 149.86 153.67 0)
 			(effects
@@
 			)
 		)
-		(pin "MP"
+		(pin "1"
 		)
 		(instances
@@
 	)
 	(symbol
-		(lib_id "Mechanical:MountingHole_Pad_MP")
+		(lib_id "Mechanical:MountingHole_Pad")
 		(at 134.62 153.67 180)
 		(unit 1)
@@
 			)
 		)
-		(property "Footprint" "MountingHole:MountingHole_2.5mm"
+		(property "Footprint" "MountingHole:MountingHole_2.5mm_Pad_Via"
 			(at 134.62 153.67 0)
 			(effects
@@
 			)
 		)
-		(property "Description" "Mounting Hole with connection as pad named MP"
+		(property "Description" "Mounting Hole with connection"
 			(at 134.62 153.67 0)
 			(effects
@@
 			)
 		)
-		(pin "MP"
+		(pin "1"
 		)
 		(instances

Commit message: Finished Layout V1
Changed lines of the file:
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@@
 	)
 	(global_label "SN_2"
-		(shape passive)
+		(shape output)
 		(at 127 106.68 180)
 		(fields_autoplaced yes)
@@
 		)
 		(property "Intersheetrefs" "${INTERSHEET_REFS}"
-			(at 120.409 106.68 0)
+			(at 119.2977 106.68 0)
 			(effects
 				(font
@@
 	)
 	(global_label "SN_1"
-		(shape passive)
+		(shape output)
 		(at 34.29 105.41 180)
 		(fields_autoplaced yes)
@@
 		)
 		(property "Intersheetrefs" "${INTERSHEET_REFS}"
-			(at 27.699 105.41 0)
+			(at 26.5877 105.41 0)
 			(effects
 				(font
@@
 	)
 	(global_label "SP_2"
-		(shape passive)
+		(shape output)
 		(at 127 121.92 180)
 		(fields_autoplaced yes)
@@
 		)
 		(property "Intersheetrefs" "${INTERSHEET_REFS}"
-			(at 120.4695 121.92 0)
+			(at 119.3582 121.92 0)
 			(effects
 				(font
@@
 	)
 	(global_label "SP_1"
-		(shape passive)
+		(shape output)
 		(at 34.29 120.65 180)
 		(fields_autoplaced yes)
@@
 		)
 		(property "Intersheetrefs" "${INTERSHEET_REFS}"
-			(at 27.7595 120.65 0)
-			(effects
-				(font
+			(at 26.6482 120.65 0)
+			(effects
+				(font

Commit message: PCB V2, CAD V3 & Code
Parts:
- C401, C405, C408: footprint Capacitor_SMD:C_0402_1005Metric -> Capacitor_SMD:C_0805_2012Metric
Changed lines of the file:
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@@
 			)
 		)
-		(property "Footprint" "Capacitor_SMD:C_0402_1005Metric"
+		(property "Footprint" "Capacitor_SMD:C_0805_2012Metric"
 			(at 67.31 52.07 0)
 			(effects
@@
 			)
 		)
-		(property "Footprint" "Capacitor_SMD:C_0402_1005Metric"
+		(property "Footprint" "Capacitor_SMD:C_0805_2012Metric"
 			(at 160.02 53.34 0)
 			(effects
@@
 			)
 		)
-		(property "Footprint" "Capacitor_SMD:C_0402_1005Metric"
+		(property "Footprint" "Capacitor_SMD:C_0805_2012Metric"
 			(at 246.38 54.61 0)
 			(effects

Commit message: PCB_V2
Parts:
- Q401, Q402, Q403, Q404, Q405, Q406: value IRFH7440TRPBF -> FH4008GS; footprint IRFH7440TRPBF:IRFH7440TRPBF -> Package_DFN_QFN:PQFN-8-EP_6x5mm_P1.27mm_Generic
- R404, R409, R414: value 68k -> 100k
Other:
- note added: "Adapted for 36V max reading"
- note added: "BIGGER MOTOR - 22ohm"
- company: (none) -> ANGEL PELEGRY VELASCO
