File: Hardware/ESP32_Motor_Controller/POWER_MOSFET.kicad_sch (KiCad schematic)
At the start: 38 parts, among them Q401 FH4008GS, Q402 FH4008GS, Q403 FH4008GS, Q404 FH4008GS, Q405 FH4008GS, Q406 FH4008GS

Commit message: Adapted for Main Robot
Parts:
- C401, C405, C408: value 2.2 uF -> 2.2uF
Changed lines of the file:
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@@
 			"cgB2AHYAOQB2AFAAegBrADUAVQBIAEEAQQBBAEEAQQBHAEEARABmAGYAcgAwAHUAZgB2AHUAdQA4"
 			"AFYASgBYAGwANQBlAFoAbQBhAG0AcgBEAHkAdwBCAGcAbwBkAFIANgBaADQAUABNAGYAYgAyADMA"
-			"dgBoAHcAbwBXAFMAcwBnAEEAQQ=="
+			"dgBoAHcAbwBXAFMAcwBnAEEAQQBaAEgAVgAzAGQAMwAvAG8AbwBZAGMAawA1AGcARQBBAEEAQQBB"
+			"AEEAYQBNAEcAdgBmAHYAVwByAG4AagAxADcAbQBnAC8AYgAyAHQAbwArACsATwBDAEQAagBvADQA"
+			"TwBpAFoARgBnAEkAUQBvAGQAeAAxAEYAZABYAGIAMQBxADEAUwBwAHgATQBtAFgASwBsAFAARAB3"
+			"AGMARgBsADUAQQBBAEEAQQBBAEEAQQBhAE0AVwB6AFkAcwBLAFMAawBKAEgARwB5AGQAZQB2AFcA"
+			"cwByAEkAeQBXAFgAbABnAE8AUQBvAGQAeAA3AEYAdQAzAGIAcQBLAGkAZwBwAHgAOAB1AGkAagBq"
+			"ADgAbwBLAEEAdwBBAEEAQQBBAEQAUQBsAEUAYwBmAGYAZABUAFoAKwBkADgAbABRAEYAMQBkADMA"
+			"ZgBmAGYAZgB5ADgAeABEAHkAeABFAG8AZQBNAGcAVABDAGIAVABwADUAOQArAEsAawA2AEcARABS"
+			"AHMAMgBjACsAWgBNAFcAWABrAEEAQQBBAEEAQQBBAEoAbwB5AGUAZgBMAGsAcwBXAFAASABpAHAA"
+			"TgB2AHYAdgBtAG0AbwBhAEYAQgBWAGgANQBZAGkARQBMAEgAUQBlAFQAbQA1AHUAYgBrADUASQBp"
+			"AFQAQgBRAHMAVwA5AE8ANwBkAFcAMQBZAGUAQQBBAEEAQQBBAEkAQwBtAGQATwB2AFcAYgBlAEgA"
+			"QwBoAGUASwBrAHUATABoADQAKwAvAGIAdABrAHUATABBAFUAaABRADYARAB1AEwAVABUAHoAOAAx"
+			"AG0AVQB6AG0AdwAyADcAZAB1AHQAMQAvAC8ALwAwAFMAOAB3AEEAQQBBAEEAQQBBAHQARwBiAHUA"
+			"MwBMAGwAKwBmAG4ANwBtAHcANAA2AE8AagBvADgALwAvAHAAaQBsAGsAZQAwAFUAaABZADQAagBP"
+			"AEgAMwA2ADkASgBvADEAYQA4AFQASgA5AE8AbgBUAFEAMABKAEMAWgBPAFUAQgBBAEEAQQBBAEEA"
+			"RwBqAFEANABNAEcARABiADcALwA5AGQAbgBHAFMAbgBwADUAZQBXAEYAZwBvAEsAdwA4AHMAUQBh"
+			"AEgAagBDAEQAWgBzADIASABEADIANwBGAGwAeAB3AG4ATABJAEEAQQBBAEEAQQBJAEEAcgAvAGYA"
+			"YQAzAHYAMwBWADEAZABUAFUAZgBOAGoAUQAwAEwARgB1ADIAVABHAEkAZQBkAEIAbQBGAGoAaQBQ"
+			"ADQAOABzAHMAdgB4AGMATwBBAGcASQBBAFoATQAyAFoASQB5AGcASQBBAEEAQQBBAEEAMABLADQA"
+			"SgBFAHkAYQBNAEcAVABOAEcAbg=="
 		)
 	)
@@
 			)
 		)
-		(property "Value" "2.2 uF"
+		(property "Value" "2.2uF"
 			(at 69.85 53.3462 0)
 			(effects
@@
 			)
 		)
-		(property "Value" "2.2 uF"
+		(property "Value" "2.2uF"
 			(at 162.56 54.6162 0)
 			(effects
@@
 			)
 		)
-		(property "Value" "2.2 uF"
+		(property "Value" "2.2uF"
 			(at 248.92 55.8862 0)
 			(effects
