File: Hardware/ESP32_Motor_Controller/GATE DRIVER [3].kicad_sch (KiCad schematic)
At the start: 44 parts, among them U301 DRV8302DCAR

Commit message: Adapted for Main Robot
Parts:
- C319: value 12uH -> 22uF
Changed lines of the file:
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@@
 			"NQBVAEgAQQBBAEEAQQBBAEcAQQBEAGYAZgByADAAdQBmAHYAdQB1ADgAVgBKAFgAbAA1AGUAWgBt"
 			"AGEAbQByAEQAeQB3AEIAZwBvAGQAUgA2AFoANABQAE0AZgBiADIAMwB2AGgAdwBvAFcAUwBzAGcA"
-			"QQBBAEEAQQBBAEEAYgBPAGYAKw=="
+			"QQBBAEEAQQBBAEEAYgBPAGYAKwBaAEgAVgAzAGQAMwAvAG8AbwBZAGMAawA1AGcARQBBAEEAQQBB"
+			"AEEAYQBNAEcAdgBmAHYAVwByAG4AagAxADcAbQBnAC8AYgAyAHQAbwArACsATwBDAEQAagBvADQA"
+			"TwBpAFoARgBnAEkAUQBvAGQAeAAxAEYAZABYAGIAMQBxADEAUwBwAHgATQBtAFgASwBsAFAARAB3"
+			"AGMARgBsADUAQQBBAEEAQQBBAEEAQQBhAE0AVwB6AFkAcwBLAFMAawBKAEgARwB5AGQAZQB2AFcA"
+			"cwByAEkAeQBXAFgAbABnAE8AUQBvAGQAeAA3AEYAdQAzAGIAcQBLAGkAZwBwAHgAOAB1AGkAagBq"
+			"ADgAbwBLAEEAdwBBAEEAQQBBAEQAUQBsAEUAYwBmAGYAZABUAFoAKwBkADgAbABRAEYAMQBkADMA"
+			"ZgBmAGYAZgB5ADgAeABEAHkAeABFAG8AZQBNAGcAVABDAGIAVABwADUAOQArAEsAawA2AEcARABS"
+			"AHMAMgBjACsAWgBNAFcAWABrAEEAQQBBAEEAQQBBAEoAbwB5AGUAZgBMAGsAcwBXAFAASABpAHAA"
+			"TgB2AHYAdgBtAG0AbwBhAEYAQgBWAGgANQBZAGkARQBMAEgAUQBlAFQAbQA1AHUAYgBrADUASQBp"
+			"AFQAQgBRAHMAVwA5AE8ANwBkAFcAMQBZAGUAQQBBAEEAQQBBAEkAQwBtAGQATwB2AFcAYgBlAEgA"
+			"QwBoAGUASwBrAHUATABoADQAKwAvAGIAdABrAHUATABBAFUAaABRADYARAB1AEwAVABUAHoAOAAx"
+			"AG0AVQB6AG0AdwAyADcAZAB1AHQAMQAvAC8ALwAwAFMAOAB3AEEAQQBBAEEAQQBBAHQARwBiAHUA"
+			"MwBMAGwAKwBmAG4ANwBtAHcANAA2AE8AagBvADgALwAvAHAAaQBsAGsAZQAwAFUAaABZADQAagBP"
+			"AEgAMwA2ADkASgBvADEAYQA4AFQASgA5AE8AbgBUAFEAMABKAEMAWgBPAFUAQgBBAEEAQQBBAEEA"
+			"RwBqAFEANABNAEcARABiADcALwA5AGQAbgBHAFMAbgBwADUAZQBXAEYAZwBvAEsAdwA4AHMAUQBh"
+			"AEgAagBDAEQAWgBzADIASABEADIANwBGAGwAeAB3AG4ATABJAEEAQQBBAEEAQQBJAEEAcgAvAGYA"
+			"YQAzAHYAMwBWADEAZABUAFUAZgBOAGoAUQAwAEwARgB1ADIAVABHAEkAZQBkAEIAbQBGAGoAaQBQ"
+			"ADQAOABzAHMAdgB4AGMATwBBAGcASQBBAFoATQAyAFoASQB5AGcASQBBAEEAQQBBAEEAMABLADQA"
+			"SgBFAHkAYQBNAEcAVABOAEcAbg=="
 		)
 	)
@@
 			)
 		)
-		(column_widths 16.51 7.62 9.525 7.62)
+		(column_widths 16.51 7.62 9.525 12.7)
 		(row_heights 3.81 3.81 3.81 3.81 3.81 3.81 3.81)
 		(cells
@@
 				(exclude_from_sim no)
 				(at 50.8 16.51 0)
-				(size 7.62 3.81)
+				(size 12.7 3.81)
 				(margins 0.9525 0.9525 0.9525 0.9525)
 				(span 1 1)
@@
 				(exclude_from_sim no)
 				(at 50.8 20.32 0)
-				(size 7.62 3.81)
+				(size 12.7 3.81)
 				(margins 0.9525 0.9525 0.9525 0.9525)
 				(span 1 1)
@@
 				)
 			)
-			(table_cell "42uH"
+			(table_cell "12uH"
 				(exclude_from_sim no)
 				(at 50.8 24.13 0)
-				(size 7.62 3.81)
+				(size 12.7 3.81)
 				(margins 0.9525 0.9525 0.9525 0.9525)
 				(span 1 1)
@@
 				)
 			)
-			(table_cell "47uF"
+			(table_cell "22uF x 2"
 				(exclude_from_sim no)
 				(at 50.8 27.94 0)
-				(size 7.62 3.81)
+				(size 12.7 3.81)
 				(margins 0.9525 0.9525 0.9525 0.9525)
 				(span 1 1)
@@
 				)
 			)
-			(table_cell "280k"
+			(table_cell "21.5k"
 				(exclude_from_sim no)
 				(at 50.8 31.75 0)
-				(size 7.62 3.81)
+				(size 12.7 3.81)
 				(margins 0.9525 0.9525 0.9525 0.9525)
 				(span 1 1)
@@
 				)
 			)
-			(table_cell "1nF"
+			(table_cell "6.8nF"
 				(exclude_from_sim no)
 				(at 50.8 35.56 0)
-				(size 7.62 3.81)
+				(size 12.7 3.81)
 				(margins 0.9525 0.9525 0.9525 0.9525)
 				(span 1 1)
@@
 				)
 			)
-			(table_cell ">5pF"
+			(table_cell "27pF"
 				(exclude_from_sim no)
 				(at 50.8 39.37 0)
-				(size 7.62 3.81)
+				(size 12.7 3.81)
 				(margins 0.9525 0.9525 0.9525 0.9525)
 				(span 1 1)
@@
 			)
 		)
-		(property "Value" "12uH"
+		(property "Value" "22uF"
 			(at 80.01 71.1262 0)
 			(effects
